Commit message: 

File: elf2_dof25/urdf/elf2_dof25.urdf (robot description, URDF)
Before this commit: robot elf2_dof25, 26 links, 25 joints
Links:
- link base_link: geometry collision mesh filename=meshes/base_link.STL; visual mesh filename=meshes/base_link.STL
- link l_ankle_x_link: geometry collision mesh filename=meshes/l_ankle_x_link.STL; visual mesh filename=meshes/l_ankle_x_link.STL
- link l_ankle_y_link: geometry collision mesh filename=meshes/l_ankle_y_link.STL; visual mesh filename=meshes/l_ankle_y_link.STL
- link l_elb_y_link: geometry collision mesh filename=meshes/l_elb_y_link.STL; visual mesh filename=meshes/l_elb_y_link.STL
- link l_elb_z_link: geometry collision mesh filename=meshes/l_elb_z_link.STL; visual mesh filename=meshes/l_elb_z_link.STL
- link l_hip_x_link: geometry collision mesh filename=meshes/l_hip_x_link.STL; visual mesh filename=meshes/l_hip_x_link.STL
- link l_hip_y_link: geometry collision mesh filename=meshes/l_hip_y_link.STL; visual mesh filename=meshes/l_hip_y_link.STL
- link l_hip_z_link: geometry collision mesh filename=meshes/l_hip_z_link.STL; visual mesh filename=meshes/l_hip_z_link.STL
- link l_knee_y_link: geometry collision mesh filename=meshes/l_knee_y_link.STL; visual mesh filename=meshes/l_knee_y_link.STL
- link l_shld_x_link: geometry collision mesh filename=meshes/l_shld_x_link.STL; visual mesh filename=meshes/l_shld_x_link.STL
- link l_shld_y_link: geometry collision mesh filename=meshes/l_shld_y_link.STL; visual mesh filename=meshes/l_shld_y_link.STL
- link l_shld_z_link: geometry collision mesh filename=meshes/l_shld_z_link.STL; visual mesh filename=meshes/l_shld_z_link.STL
- link r_ankle_x_link: geometry collision mesh filename=meshes/r_ankle_x_link.STL; visual mesh filename=meshes/r_ankle_x_link.STL
- link r_ankle_y_link: geometry collision mesh filename=meshes/r_ankle_y_link.STL; visual mesh filename=meshes/r_ankle_y_link.STL
- link r_elb_y_link: geometry collision mesh filename=meshes/r_elb_y_link.STL; visual mesh filename=meshes/r_elb_y_link.STL
- link r_elb_z_link: geometry collision mesh filename=meshes/r_elb_z_link.STL; visual mesh filename=meshes/r_elb_z_link.STL
- link r_hip_x_link: geometry collision mesh filename=meshes/r_hip_x_link.STL; visual mesh filename=meshes/r_hip_x_link.STL
- link r_hip_y_link: geometry collision mesh filename=meshes/r_hip_y_link.STL; visual mesh filename=meshes/r_hip_y_link.STL
- link r_hip_z_link: geometry collision mesh filename=meshes/r_hip_z_link.STL; visual mesh filename=meshes/r_hip_z_link.STL
- link r_knee_y_link: geometry collision mesh filename=meshes/r_knee_y_link.STL; visual mesh filename=meshes/r_knee_y_link.STL
- link r_shld_x_link: geometry collision mesh filename=meshes/r_shld_x_link.STL; visual mesh filename=meshes/r_shld_x_link.STL
- link r_shld_y_link: geometry collision mesh filename=meshes/r_shld_y_link.STL; visual mesh filename=meshes/r_shld_y_link.STL
- link r_shld_z_link: geometry collision mesh filename=meshes/r_shld_z_link.STL; visual mesh filename=meshes/r_shld_z_link.STL
- link waist_x_link: geometry collision mesh filename=meshes/waist_x_link.STL; visual mesh filename=meshes/waist_x_link.STL
- link waist_y_link: geometry collision mesh filename=meshes/waist_y_link.STL; visual mesh filename=meshes/waist_y_link.STL
- link waist_z_link: geometry collision mesh filename=meshes/waist_z_link.STL; visual mesh filename=meshes/waist_z_link.STL
